Commit message: added irbt4004 reversed

File: abb_irbt4004_support/urdf/irbt4004r_macro.xacro (robot description, xacro)
@@ -4,20 +4,19 @@
 <robot xmlns:xacro="http://ros.org/wiki/xacro">
   <xacro:include filename="$(find abb_resources)/urdf/common_materials.xacro"/>
-  <xacro:macro name="abb_irbt4004" params="prefix">
-    <!-- link zero-->
-<!--    <link name="${prefix}world"/>-->
+  <xacro:macro name="abb_irbt4004r" params="prefix">
     <!-- link list -->
-    <link name="${prefix}track_left"> <!--track_start-->
+    <!--Right section-->
+    <link name="${prefix}track_right">
       <visual>
-        <origin xyz="0 0 0" rpy="0 0 0"/>
+        <origin xyz="-2.5 0 0" rpy="0 0 0"/>
         <geometry>
-          <mesh filename="package://abb_irbt4004_support/meshes/irbt4004/visual/Track_Start.stl"/>
+          <mesh filename="package://abb_irbt4004_support/meshes/irbt4004/visual/Track_End.stl"/>
         </geometry>
         <xacro:material_abb_orange />
       </visual>
       <collision>
-        <origin xyz="0 0 0" rpy="0 0 0"/>
+        <origin xyz="-2.5 0 0" rpy="0 0 0"/>
         <geometry>
-          <mesh filename="package://abb_irbt4004_support/meshes/irbt4004/collision/Track_Start.stl"/>
+          <mesh filename="package://abb_irbt4004_support/meshes/irbt4004/collision/Track_End.stl"/>
         </geometry>
         <xacro:material_abb_orange />
@@ -26,5 +25,5 @@
     <link name="${prefix}track_mid_1">
       <visual>
-        <origin xyz="0 0 0" rpy="0 0 0"/>
+        <origin xyz="-2.5 0 0" rpy="0 0 0"/>
         <geometry>
           <mesh filename="package://abb_irbt4004_support/meshes/irbt4004/visual/Track_Mid.stl"/>
@@ -33,5 +32,5 @@
       </visual>
       <collision>
-        <origin xyz="0 0 0" rpy="0 0 0"/>
+        <origin xyz="-2.5 0 0" rpy="0 0 0"/>
         <geometry>
           <mesh filename="package://abb_irbt4004_support/meshes/irbt4004/collision/Track_Mid.stl"/>
@@ -42,5 +41,5 @@
     <link name="${prefix}track_mid_2">
       <visual>
-        <origin xyz="0 0 0" rpy="0 0 0"/>
+        <origin xyz="-2.5 0 0" rpy="0 0 0"/>
         <geometry>
           <mesh filename="package://abb_irbt4004_support/meshes/irbt4004/visual/Track_Mid.stl"/>
@@ -49,5 +48,5 @@
       </visual>
       <collision>
-        <origin xyz="0 0 0" rpy="0 0 0"/>
+        <origin xyz="-2.5 0 0" rpy="0 0 0"/>
         <geometry>
           <mesh filename="package://abb_irbt4004_support/meshes/irbt4004/collision/Track_Mid.stl"/>
@@ -58,5 +57,5 @@
     <link name="${prefix}track_mid_3">
       <visual>
-        <origin xyz="0 0 0" rpy="0 0 0"/>
+        <origin xyz="-2.5 0 0" rpy="0 0 0"/>
         <geometry>
           <mesh filename="package://abb_irbt4004_support/meshes/irbt4004/visual/Track_Mid.stl"/>
@@ -65,5 +64,5 @@
       </visual>
       <collision>
-        <origin xyz="0 0 0" rpy="0 0 0"/>
+        <origin xyz="-2.5 0 0" rpy="0 0 0"/>
         <geometry>
           <mesh filename="package://abb_irbt4004_support/meshes/irbt4004/collision/Track_Mid.stl"/>
@@ -72,42 +71,24 @@
       </collision>
     </link>
-    <!--Right section-->
-<!--    <link name="${prefix}track_right">
+    <link name="${prefix}track_mid_4">
       <visual>
-        <origin xyz="0 0 0" rpy="0 0 0"/>
+        <origin xyz="-2.5 0 0" rpy="0 0 0"/>
         <geometry>
-          <mesh filename="package://abb_irbt4004_support/meshes/irbt4004/visual/Track_End.stl"/>
+          <mesh filename="package://abb_irbt4004_support/meshes/irbt4004/visual/Track_Mid.stl"/>
         </geometry>
         <xacro:material_abb_orange />
       </visual>
       <collision>
-        <origin xyz="0 0 0" rpy="0 0 0"/>
+        <origin xyz="-2.5 0 0" rpy="0 0 0"/>
         <geometry>
-          <mesh filename="package://abb_irbt4004_support/meshes/irbt4004/collision/Track_End.stl"/>
+          <mesh filename="package://abb_irbt4004_support/meshes/irbt4004/collision/Track_Mid.stl"/>
         </geometry>
         <xacro:material_abb_orange />
       </collision>
-    </link>-->
-    <!--Left carriage-->
+    </link>
+    <!--Right carriage-->
     <link name="${prefix}carriage">
       <visual>
-      <origin xyz="0 0 0" rpy="0 0 0"/>
-        <geometry>
-          <mesh filename="package://abb_irbt4004_support/meshes/irbt4004/visual/Carriage_left.stl"/>
-        </geometry>
-        <xacro:material_abb_dark_gray />
-      </visual>
-      <collision>
-        <origin xyz="0 0 0" rpy="0 0 0"/>
-        <geometry>
-          <mesh filename="package://abb_irbt4004_support/meshes/irbt4004/collision/Carriage_left.stl"/>
-        </geometry>
-        <xacro:material_abb_dark_gray />
-      </collision>
-    </link>
-    <!--Right carriage-->
-<!--    <link name="${prefix}carriage2">
-      <visual>
-      <origin xyz="0 0 0" rpy="0 0 0"/>
+      <origin xyz="-0.5 0 0" rpy="0 0 0"/>
         <geometry>
           <mesh filename="package://abb_irbt4004_support/meshes/irbt4004/visual/Carriage_right.stl"/>
@@ -116,5 +97,5 @@
       </visual>
       <collision>
-        <origin xyz="0 0 0" rpy="0 0 0"/>
+        <origin xyz="-0.5 0 0" rpy="0 0 0"/>
         <geometry>
           <mesh filename="package://abb_irbt4004_support/meshes/irbt4004/collision/Carriage_right.stl"/>
@@ -122,21 +103,26 @@
         <xacro:material_abb_dark_gray />
       </collision>
-    </link>-->
+    </link>
     <!-- end of link list -->
     <!-- joint list -->
     <joint name="${prefix}fixed_track_mid_1" type="fixed">
-      <parent link="${prefix}track_left"/>
+      <parent link="${prefix}track_right"/>
       <child link="${prefix}track_mid_1"/>
-      <origin xyz="0.000 0.000 0.000" rpy="0 0 0"/>
+      <origin xyz="-1.000 0.000 0.000" rpy="0 0 0"/>
     </joint>
     <joint name="${prefix}fixed_track_mid_2" type="fixed">
       <parent link="${prefix}track_mid_1"/>
       <child link="${prefix}track_mid_2"/>
-      <origin xyz="1.000 0.000 0.000" rpy="0 0 0"/>
+      <origin xyz="-1.000 0.000 0.000" rpy="0 0 0"/>
     </joint>
     <joint name="${prefix}fixed_track_mid_3" type="fixed">
       <parent link="${prefix}track_mid_2"/>
       <child link="${prefix}track_mid_3"/>
-      <origin xyz="1.000 0.000 0.000" rpy="0 0 0"/>
+      <origin xyz="-1.000 0.000 0.000" rpy="0 0 0"/>
+    </joint>
+    <joint name="${prefix}fixed_track_mid_4" type="fixed">
+      <parent link="${prefix}track_mid_3"/>
+      <child link="${prefix}track_mid_4"/>
+      <origin xyz="-1.000 0.000 0.000" rpy="0 0 0"/>
     </joint>
     <!--Track end-->
@@ -148,8 +134,8 @@
     <!--Left carriage-->
     <joint name="${prefix}joint_carriage" type="prismatic">
-      <parent link="${prefix}track_left"/>
+      <parent link="${prefix}track_right"/>
       <child link="${prefix}carriage"/>
-      <origin xyz="0 0 0" rpy="0 0 0"/>
-      <axis xyz="1 0 0"/>
+      <origin xyz="-0.1 0 0" rpy="0 0 0"/>
+      <axis xyz="-1 0 0"/>
       <limit effort="0" lower="0.000" upper="3.900" velocity="2.000"/> <!-- Product specification - IRBT 4004/6004/7004 -->
     </joint>
