Commit message: irbt4004 update

File: abb_irbt4004_support/urdf/irbt4004_macro.xacro (robot description, xacro)
@@ -6,5 +6,5 @@
 <!--    <link name="${prefix}world"/>-->
     <!-- link list -->
-    <link name="${prefix}base_link"> <!--track_start-->
+    <link name="${prefix}track_left"> <!--track_start-->
       <visual>
         <origin xyz="0 0 0" rpy="0 0 0"/>
@@ -70,10 +70,10 @@
       </collision>
     </link>
-    <!-- no end section
-    <link name="${prefix}track_end">
+    <!--Right section-->
+<!--    <link name="${prefix}track_right">
       <visual>
         <origin xyz="0 0 0" rpy="0 0 0"/>
         <geometry>
-          <mesh filename="package://abb_irbt4004_support/meshes/irb4400/visual/Track_End.stl"/>
+          <mesh filename="package://abb_irbt4004_support/meshes/irbt4004/visual/Track_End.stl"/>
         </geometry>
         <xacro:material_abb_orange />
@@ -82,13 +82,13 @@
         <origin xyz="0 0 0" rpy="0 0 0"/>
         <geometry>
-          <mesh filename="package://abb_irbt4004_support/meshes/irb4400/collision/Track_End.stl"/>
+          <mesh filename="package://abb_irbt4004_support/meshes/irbt4004/collision/Track_End.stl"/>
         </geometry>
         <xacro:material_abb_orange />
       </collision>
-    </link>
-    -->
+    </link>-->
+    <!--Left carriage-->
     <link name="${prefix}carriage">
       <visual>
-        <origin xyz="0 0 0" rpy="0 0 0"/>
+      <origin xyz="0 0 0" rpy="0 0 0"/>
         <geometry>
           <mesh filename="package://abb_irbt4004_support/meshes/irbt4004/visual/Carriage_left.stl"/>
@@ -104,8 +104,25 @@
       </collision>
     </link>
+    <!--Right carriage-->
+<!--    <link name="${prefix}carriage2">
+      <visual>
+      <origin xyz="0 0 0" rpy="0 0 0"/>
+        <geometry>
+          <mesh filename="package://abb_irbt4004_support/meshes/irbt4004/visual/Carriage_right.stl"/>
+        </geometry>
+        <xacro:material_abb_dark_gray />
+      </visual>
+      <collision>
+        <origin xyz="0 0 0" rpy="0 0 0"/>
+        <geometry>
+          <mesh filename="package://abb_irbt4004_support/meshes/irbt4004/collision/Carriage_right.stl"/>
+        </geometry>
+        <xacro:material_abb_dark_gray />
+      </collision>
+    </link>-->
     <!-- end of link list -->
     <!-- joint list -->
     <joint name="${prefix}fixed_track_mid_1" type="fixed">
-      <parent link="${prefix}base_link"/>
+      <parent link="${prefix}track_left"/>
       <child link="${prefix}track_mid_1"/>
       <origin xyz="0.000 0.000 0.000" rpy="0 0 0"/>
@@ -121,18 +138,27 @@
       <origin xyz="1.000 0.000 0.000" rpy="0 0 0"/>
     </joint>
-    <!-- no end section
-    <joint name="${prefix}fixed_track_end" type="fixed">
+    <!--Track end-->
+<!--    <joint name="${prefix}fixed_track_right" type="fixed">
       <parent link="${prefix}track_mid_3"/>
-      <child link="${prefix}track_end"/>
+      <child link="${prefix}track_right"/>
       <origin xyz="1.000 0.000 0.000" rpy="0 0 0"/>
-    </joint>
-    -->
+    </joint>-->
+    <!--Left carriage-->
     <joint name="${prefix}joint_carriage" type="prismatic">
-      <parent link="${prefix}base_link"/>
+      <parent link="${prefix}track_left"/>
       <child link="${prefix}carriage"/>
+      <origin xyz="0 0 0" rpy="0 0 0"/>
       <axis xyz="1 0 0"/>
       <limit effort="0" lower="0.000" upper="3.700" velocity="2.000"/> <!-- Product specification - IRBT 4004/6004/7004 -->
     </joint>
-    <!-- offset to center base plate for robot mounting position
+    <!--Right carriage-->
+<!--    <joint name="${prefix}joint_carriage2" type="prismatic">
+      <parent link="${prefix}track_right"/>
+      <child link="${prefix}carriage2"/>
+      <origin xyz="0 0 0" rpy="0 0 0"/>
+      <axis xyz="-1 0 0"/>
+      <limit effort="0" lower="0.000" upper="3.700" velocity="2.000"/>
+    </joint>-->
+<!-- offset to center base plate for robot mounting position
     <joint name="${prefix}fixed_base_link" type="fixed">
       <parent link="${prefix}carriage"/>
@@ -141,11 +167,4 @@
     </joint>-->
     <!-- end of joint list -->
-<!-- ROS base_link to ABB World Coordinates transform -->
-    <link name="${prefix}base" />
-    <joint name="${prefix}base_link-base" type="fixed">
-      <origin xyz="0 0 0" rpy="0 0 0"/>
-      <parent link="${prefix}base_link"/>
-      <child link="${prefix}base"/>
-    </joint>
   </xacro:macro>
 </robot>

Commit message: irbt4004 - added robot interface point

File: abb_irbt4004_support/urdf/irbt4004_macro.xacro (robot description, xacro)
@@ -5,6 +5,4 @@
   <xacro:include filename="$(find abb_resources)/urdf/common_materials.xacro"/>
   <xacro:macro name="abb_irbt4004" params="prefix">
-    <!-- link zero-->
-<!--    <link name="${prefix}world"/>-->
     <!-- link list -->
     <link name="${prefix}track_left"> <!--track_start-->
@@ -73,5 +71,5 @@
     </link>
     <!--Right section-->
-<!--    <link name="${prefix}track_right">
+    <!--<link name="${prefix}track_right">
       <visual>
         <origin xyz="0 0 0" rpy="0 0 0"/>
@@ -107,5 +105,5 @@
     </link>
     <!--Right carriage-->
-<!--    <link name="${prefix}carriage2">
+    <!--<link name="${prefix}carriage2">
       <visual>
       <origin xyz="0 0 0" rpy="0 0 0"/>
@@ -123,4 +121,5 @@
       </collision>
     </link>-->
+    <link name="${prefix}carriage_interface"/>
     <!-- end of link list -->
     <!-- joint list -->
@@ -141,10 +140,10 @@
     </joint>
     <!--Track end-->
-<!--    <joint name="${prefix}fixed_track_right" type="fixed">
+    <!--<joint name="${prefix}fixed_track_right" type="fixed">
       <parent link="${prefix}track_mid_3"/>
       <child link="${prefix}track_right"/>
       <origin xyz="1.000 0.000 0.000" rpy="0 0 0"/>
     </joint>-->
-    <!--Left carriage-->
+    <!--carriage-->
     <joint name="${prefix}joint_carriage" type="prismatic">
       <parent link="${prefix}track_left"/>
@@ -154,18 +153,10 @@
       <limit effort="0" lower="0.000" upper="3.900" velocity="2.000"/> <!-- Product specification - IRBT 4004/6004/7004 -->
     </joint>
-    <!--Right carriage-->
-<!--    <joint name="${prefix}joint_carriage2" type="prismatic">
-      <parent link="${prefix}track_right"/>
-      <child link="${prefix}carriage2"/>
-      <origin xyz="0 0 0" rpy="0 0 0"/>
-      <axis xyz="-1 0 0"/>
-      <limit effort="0" lower="0.000" upper="3.700" velocity="2.000"/>
-    </joint>-->
-<!-- offset to center base plate for robot mounting position
-    <joint name="${prefix}fixed_base_link" type="fixed">
+    <!-- Robot interface point -->
+    <joint name="${prefix}carriage_interface_link" type="fixed">
       <parent link="${prefix}carriage"/>
-      <child link="${prefix}base_link"/>
-      <origin xyz="0.3955 0.560 0.3745" rpy="0 0 1.57079632"/>
-    </joint>-->
+      <child link="${prefix}carriage_interface"/>
+      <origin xyz="0.3955 0.560 0.3745" rpy="0 0 1.57079632" />
+    </joint>
     <!-- end of joint list -->
   </xacro:macro>

File: abb_irbt4004_support/urdf/irbt4004r_macro.xacro (robot description, xacro)
@@ -6,5 +6,4 @@
   <xacro:macro name="abb_irbt4004r" params="prefix">
     <!-- link list -->
-    <!--Right section-->
     <link name="${prefix}track_right">
       <visual>
@@ -104,4 +103,5 @@
       </collision>
     </link>
+    <link name="${prefix}carriage_interface"/>
     <!-- end of link list -->
     <!-- joint list -->
@@ -126,11 +126,5 @@
       <origin xyz="-1.000 0.000 0.000" rpy="0 0 0"/>
     </joint>
-    <!--Track end-->
-<!--    <joint name="${prefix}fixed_track_right" type="fixed">
-      <parent link="${prefix}track_mid_3"/>
-      <child link="${prefix}track_right"/>
-      <origin xyz="1.000 0.000 0.000" rpy="0 0 0"/>
-    </joint>-->
-    <!--Left carriage-->
+    <!--carriage-->
     <joint name="${prefix}joint_carriage" type="prismatic">
       <parent link="${prefix}track_right"/>
@@ -140,18 +134,10 @@
       <limit effort="0" lower="0.000" upper="3.900" velocity="2.000"/> <!-- Product specification - IRBT 4004/6004/7004 -->
     </joint>
-    <!--Right carriage-->
-<!--    <joint name="${prefix}joint_carriage2" type="prismatic">
-      <parent link="${prefix}track_right"/>
-      <child link="${prefix}carriage2"/>
-      <origin xyz="0 0 0" rpy="0 0 0"/>
-      <axis xyz="-1 0 0"/>
-      <limit effort="0" lower="0.000" upper="3.700" velocity="2.000"/>
-    </joint>-->
-<!-- offset to center base plate for robot mounting position
-    <joint name="${prefix}fixed_base_link" type="fixed">
+    <!-- Robot interface point -->
+    <joint name="${prefix}carriage_interface_link" type="fixed">
       <parent link="${prefix}carriage"/>
-      <child link="${prefix}base_link"/>
-      <origin xyz="0.3955 0.560 0.3745" rpy="0 0 1.57079632"/>
-    </joint>-->
+      <child link="${prefix}carriage_interface"/>
+      <origin xyz="-0.1045 0.560 0.3745" rpy="0 0 1.57079632" />
+    </joint>
     <!-- end of joint list -->
   </xacro:macro>

Commit message: irbt4004: update mesh

File: abb_irbt4004_support/urdf/irbt4004_macro.xacro (robot description, xacro)
@@ -104,4 +104,52 @@
       </collision>
     </link>
+    <link name="${prefix}belt_loop">
+      <visual>
+      <origin xyz="0 0 0" rpy="0 0 0"/>
+        <geometry>
+          <mesh filename="package://abb_irbt4004_support/meshes/irbt4004/visual/Belt_left.stl"/>
+        </geometry>
+        <xacro:material_abb_dark_gray />
+      </visual>
+      <collision>
+        <origin xyz="0 0 0" rpy="0 0 0"/>
+        <geometry>
+          <mesh filename="package://abb_irbt4004_support/meshes/irbt4004/collision/Belt_left.stl"/>
+        </geometry>
+        <xacro:material_abb_dark_gray />
+      </collision>
+    </link>
+    <link name="${prefix}belt_1">
+      <visual>
+      <origin xyz="0 0 0" rpy="0 0 0"/>
+        <geometry>
+          <mesh filename="package://abb_irbt4004_support/meshes/irbt4004/visual/Belt_left_ext.stl"/>
+        </geometry>
+        <xacro:material_abb_dark_gray />
+      </visual>
+      <collision>
+        <origin xyz="0 0 0" rpy="0 0 0"/>
+        <geometry>
+          <mesh filename="package://abb_irbt4004_support/meshes/irbt4004/collision/Belt_left_ext.stl"/>
+        </geometry>
+        <xacro:material_abb_dark_gray />
+      </collision>
+    </link>
+    <link name="${prefix}belt_2">
+      <visual>
+      <origin xyz="0 0 0" rpy="0 0 0"/>
+        <geometry>
+          <mesh filename="package://abb_irbt4004_support/meshes/irbt4004/visual/Belt_left_ext.stl"/>
+        </geometry>
+        <xacro:material_abb_dark_gray />
+      </visual>
+      <collision>
+        <origin xyz="0 0 0" rpy="0 0 0"/>
+        <geometry>
+          <mesh filename="package://abb_irbt4004_support/meshes/irbt4004/collision/Belt_left_ext.stl"/>
+        </geometry>
+        <xacro:material_abb_dark_gray />
+      </collision>
+    </link>
     <!--Right carriage-->
     <!--<link name="${prefix}carriage2">
@@ -154,4 +202,28 @@
       <!--<limit effort="0" lower="0.000" upper="3.900" velocity="2.000"/>--> <!-- Product specification - IRBT 4004/6004/7004 -->
     </joint>
+    <joint name="${prefix}joint_belt_1" type="prismatic">
+      <parent link="${prefix}track_left"/>
+      <child link="${prefix}belt_1"/>
+      <origin xyz="0 0 0" rpy="0 0 0"/>
+      <axis xyz="1 0 0"/>
+      <limit effort="0" lower="0.000" upper="3.400" velocity="2.000"/> <!-- REDUCED LIMIT -->
+      <mimic joint="${prefix}joint_carriage" multiplier="1.0"/>
+    </joint>
+    <joint name="${prefix}joint_belt_2" type="prismatic">
+      <parent link="${prefix}track_left"/>
+      <child link="${prefix}belt_2"/>
+      <origin xyz="0 0 0" rpy="0 0 0"/>
+      <axis xyz="1 0 0"/>
+      <limit effort="0" lower="0.000" upper="3.400" velocity="2.000"/> <!-- REDUCED LIMIT -->
+      <mimic joint="${prefix}joint_carriage" multiplier="0.75"/>
+    </joint>
+    <joint name="${prefix}joint_belt_loop" type="prismatic">
+      <parent link="${prefix}track_left"/>
+      <child link="${prefix}belt_loop"/>
+      <origin xyz="0 0 0" rpy="0 0 0"/>
+      <axis xyz="1 0 0"/>
+      <limit effort="0" lower="0.000" upper="3.400" velocity="2.000"/> <!-- REDUCED LIMIT -->
+      <mimic joint="${prefix}joint_carriage" multiplier="0.5"/>
+    </joint>
     <!-- Robot interface point -->
     <joint name="${prefix}carriage_interface_link" type="fixed">
