Commit message: abb_irbt4004: update belt and collision mesh

File: abb_irbt4004_support/urdf/irbt4004_macro.xacro (robot description, xacro)
@@ -108,12 +108,28 @@
       <origin xyz="0 0 0" rpy="0 0 0"/>
         <geometry>
-          <mesh filename="package://abb_irbt4004_support/meshes/irbt4004/visual/Belt_left.stl"/>
-        </geometry>
-        <xacro:material_abb_dark_gray />
-      </visual>
-      <collision>
-        <origin xyz="0 0 0" rpy="0 0 0"/>
-        <geometry>
-          <mesh filename="package://abb_irbt4004_support/meshes/irbt4004/collision/Belt_left.stl"/>
+          <mesh filename="package://abb_irbt4004_support/meshes/irbt4004/visual/Belt_left_loop.stl"/>
+        </geometry>
+        <xacro:material_abb_dark_gray />
+      </visual>
+      <collision>
+        <origin xyz="0 0 0" rpy="0 0 0"/>
+        <geometry>
+          <mesh filename="package://abb_irbt4004_support/meshes/irbt4004/collision/Belt_left_loop.stl"/>
+        </geometry>
+        <xacro:material_abb_dark_gray />
+      </collision>
+    </link>
+    <link name="${prefix}belt_0">
+      <visual>
+      <origin xyz="0 0 0" rpy="0 0 0"/>
+        <geometry>
+          <mesh filename="package://abb_irbt4004_support/meshes/irbt4004/visual/Belt_left_ext.stl"/>
+        </geometry>
+        <xacro:material_abb_dark_gray />
+      </visual>
+      <collision>
+        <origin xyz="0 0 0" rpy="0 0 0"/>
+        <geometry>
+          <mesh filename="package://abb_irbt4004_support/meshes/irbt4004/collision/Belt_left_ext.stl"/>
         </geometry>
         <xacro:material_abb_dark_gray />
@@ -137,4 +153,36 @@
     </link>
     <link name="${prefix}belt_2">
+      <visual>
+      <origin xyz="0 0 0" rpy="0 0 0"/>
+        <geometry>
+          <mesh filename="package://abb_irbt4004_support/meshes/irbt4004/visual/Belt_left_ext.stl"/>
+        </geometry>
+        <xacro:material_abb_dark_gray />
+      </visual>
+      <collision>
+        <origin xyz="0 0 0" rpy="0 0 0"/>
+        <geometry>
+          <mesh filename="package://abb_irbt4004_support/meshes/irbt4004/collision/Belt_left_ext.stl"/>
+        </geometry>
+        <xacro:material_abb_dark_gray />
+      </collision>
+    </link>
+    <link name="${prefix}belt_3">
+      <visual>
+      <origin xyz="0 0 0" rpy="0 0 0"/>
+        <geometry>
+          <mesh filename="package://abb_irbt4004_support/meshes/irbt4004/visual/Belt_left_ext.stl"/>
+        </geometry>
+        <xacro:material_abb_dark_gray />
+      </visual>
+      <collision>
+        <origin xyz="0 0 0" rpy="0 0 0"/>
+        <geometry>
+          <mesh filename="package://abb_irbt4004_support/meshes/irbt4004/collision/Belt_left_ext.stl"/>
+        </geometry>
+        <xacro:material_abb_dark_gray />
+      </collision>
+    </link>
+    <link name="${prefix}belt_4">
       <visual>
       <origin xyz="0 0 0" rpy="0 0 0"/>
@@ -199,6 +247,21 @@
       <origin xyz="0 0 0" rpy="0 0 0"/>
       <axis xyz="1 0 0"/>
-      <limit effort="0" lower="0.000" upper="3.400" velocity="2.000"/> <!-- REDUCED LIMIT -->
-      <!--<limit effort="0" lower="0.000" upper="3.900" velocity="2.000"/>--> <!-- Product specification - IRBT 4004/6004/7004 -->
+      <limit effort="0" lower="0.000" upper="3.900" velocity="2.000"/> <!-- Product specification - IRBT 4004/6004/7004 -->
+    </joint>
+    <joint name="${prefix}joint_belt_loop" type="prismatic">
+      <parent link="${prefix}track_left"/>
+      <child link="${prefix}belt_loop"/>
+      <origin xyz="0 0 0" rpy="0 0 0"/>
+      <axis xyz="1 0 0"/>
+      <limit effort="0" lower="0.000" upper="3.900" velocity="2.000"/>
+      <mimic joint="${prefix}joint_carriage" multiplier="0.5"/>
+    </joint>
+    <joint name="${prefix}joint_belt_0" type="prismatic">
+      <parent link="${prefix}track_left"/>
+      <child link="${prefix}belt_0"/>
+      <origin xyz="0 0 0" rpy="0 0 0"/>
+      <axis xyz="1 0 0"/>
+      <limit effort="0" lower="0.000" upper="3.900" velocity="2.000"/>
+      <mimic joint="${prefix}joint_carriage" multiplier="0.5"/>
     </joint>
     <joint name="${prefix}joint_belt_1" type="prismatic">
@@ -207,22 +270,30 @@
       <origin xyz="0 0 0" rpy="0 0 0"/>
       <axis xyz="1 0 0"/>
-      <limit effort="0" lower="0.000" upper="3.400" velocity="2.000"/> <!-- REDUCED LIMIT -->
+      <limit effort="0" lower="0.000" upper="3.900" velocity="2.000"/>
+      <mimic joint="${prefix}joint_carriage" multiplier="0.625"/>
+    </joint>
+    <joint name="${prefix}joint_belt_2" type="prismatic">
+      <parent link="${prefix}track_left"/>
+      <child link="${prefix}belt_2"/>
+      <origin xyz="0 0 0" rpy="0 0 0"/>
+      <axis xyz="1 0 0"/>
+      <limit effort="0" lower="0.000" upper="3.900" velocity="2.000"/>
+      <mimic joint="${prefix}joint_carriage" multiplier="0.75"/>
+    </joint>
+    <joint name="${prefix}joint_belt_3" type="prismatic">
+      <parent link="${prefix}track_left"/>
+      <child link="${prefix}belt_3"/>
+      <origin xyz="0 0 0" rpy="0 0 0"/>
+      <axis xyz="1 0 0"/>
+      <limit effort="0" lower="0.000" upper="3.900" velocity="2.000"/>
+      <mimic joint="${prefix}joint_carriage" multiplier="0.875"/>
+    </joint>
+    <joint name="${prefix}joint_belt_4" type="prismatic">
+      <parent link="${prefix}track_left"/>
+      <child link="${prefix}belt_4"/>
+      <origin xyz="0 0 0" rpy="0 0 0"/>
+      <axis xyz="1 0 0"/>
+      <limit effort="0" lower="0.500" upper="3.900" velocity="2.000"/>
       <mimic joint="${prefix}joint_carriage" multiplier="1.0"/>
-    </joint>
-    <joint name="${prefix}joint_belt_2" type="prismatic">
-      <parent link="${prefix}track_left"/>
-      <child link="${prefix}belt_2"/>
-      <origin xyz="0 0 0" rpy="0 0 0"/>
-      <axis xyz="1 0 0"/>
-      <limit effort="0" lower="0.000" upper="3.400" velocity="2.000"/> <!-- REDUCED LIMIT -->
-      <mimic joint="${prefix}joint_carriage" multiplier="0.75"/>
-    </joint>
-    <joint name="${prefix}joint_belt_loop" type="prismatic">
-      <parent link="${prefix}track_left"/>
-      <child link="${prefix}belt_loop"/>
-      <origin xyz="0 0 0" rpy="0 0 0"/>
-      <axis xyz="1 0 0"/>
-      <limit effort="0" lower="0.000" upper="3.400" velocity="2.000"/> <!-- REDUCED LIMIT -->
-      <mimic joint="${prefix}joint_carriage" multiplier="0.5"/>
     </joint>
     <!-- Robot interface point -->

File: abb_irbt4004_support/urdf/irbt4004r_macro.xacro (robot description, xacro)
@@ -103,4 +103,100 @@
       </collision>
     </link>
+    <link name="${prefix}belt_loop">
+      <visual>
+      <origin xyz="-0.5 0 0" rpy="0 0 0"/>
+        <geometry>
+          <mesh filename="package://abb_irbt4004_support/meshes/irbt4004/visual/Belt_right_loop.stl"/>
+        </geometry>
+        <xacro:material_abb_dark_gray />
+      </visual>
+      <collision>
+        <origin xyz="-0.5 0 0" rpy="0 0 0"/>
+        <geometry>
+          <mesh filename="package://abb_irbt4004_support/meshes/irbt4004/collision/Belt_right_loop.stl"/>
+        </geometry>
+        <xacro:material_abb_dark_gray />
+      </collision>
+    </link>
+    <link name="${prefix}belt_0">
+      <visual>
+      <origin xyz="-0.5 0 0" rpy="0 0 0"/>
+        <geometry>
+          <mesh filename="package://abb_irbt4004_support/meshes/irbt4004/visual/Belt_right_ext.stl"/>
+        </geometry>
+        <xacro:material_abb_dark_gray />
+      </visual>
+      <collision>
+        <origin xyz="-0.5 0 0" rpy="0 0 0"/>
+        <geometry>
+          <mesh filename="package://abb_irbt4004_support/meshes/irbt4004/collision/Belt_right_ext.stl"/>
+        </geometry>
+        <xacro:material_abb_dark_gray />
+      </collision>
+    </link>
+    <link name="${prefix}belt_1">
+      <visual>
+      <origin xyz="-0.5 0 0" rpy="0 0 0"/>
+        <geometry>
+          <mesh filename="package://abb_irbt4004_support/meshes/irbt4004/visual/Belt_right_ext.stl"/>
+        </geometry>
+        <xacro:material_abb_dark_gray />
+      </visual>
+      <collision>
+        <origin xyz="-0.5 0 0" rpy="0 0 0"/>
+        <geometry>
+          <mesh filename="package://abb_irbt4004_support/meshes/irbt4004/collision/Belt_right_ext.stl"/>
+        </geometry>
+        <xacro:material_abb_dark_gray />
+      </collision>
+    </link>
+    <link name="${prefix}belt_2">
+      <visual>
+      <origin xyz="-0.5 0 0" rpy="0 0 0"/>
+        <geometry>
+          <mesh filename="package://abb_irbt4004_support/meshes/irbt4004/visual/Belt_right_ext.stl"/>
+        </geometry>
+        <xacro:material_abb_dark_gray />
+      </visual>
+      <collision>
+        <origin xyz="-0.5 0 0" rpy="0 0 0"/>
+        <geometry>
+          <mesh filename="package://abb_irbt4004_support/meshes/irbt4004/collision/Belt_right_ext.stl"/>
+        </geometry>
+        <xacro:material_abb_dark_gray />
+      </collision>
+    </link>
+    <link name="${prefix}belt_3">
+      <visual>
+      <origin xyz="-0.5 0 0" rpy="0 0 0"/>
+        <geometry>
+          <mesh filename="package://abb_irbt4004_support/meshes/irbt4004/visual/Belt_right_ext.stl"/>
+        </geometry>
+        <xacro:material_abb_dark_gray />
+      </visual>
+      <collision>
+        <origin xyz="-0.5 0 0" rpy="0 0 0"/>
+        <geometry>
+          <mesh filename="package://abb_irbt4004_support/meshes/irbt4004/collision/Belt_right_ext.stl"/>
+        </geometry>
+        <xacro:material_abb_dark_gray />
+      </collision>
+    </link>
+    <link name="${prefix}belt_4">
+      <visual>
+      <origin xyz="-0.5 0 0" rpy="0 0 0"/>
+        <geometry>
+          <mesh filename="package://abb_irbt4004_support/meshes/irbt4004/visual/Belt_right_ext.stl"/>
+        </geometry>
+        <xacro:material_abb_dark_gray />
+      </visual>
+      <collision>
+        <origin xyz="-0.5 0 0" rpy="0 0 0"/>
+        <geometry>
+          <mesh filename="package://abb_irbt4004_support/meshes/irbt4004/collision/Belt_right_ext.stl"/>
+        </geometry>
+        <xacro:material_abb_dark_gray />
+      </collision>
+    </link>
     <link name="${prefix}carriage_interface"/>
     <!-- end of link list -->
@@ -132,6 +228,53 @@
       <origin xyz="-0.1 0 0" rpy="0 0 0"/>
       <axis xyz="-1 0 0"/>
-      <limit effort="0" lower="0.000" upper="3.400" velocity="2.000"/> <!-- REDUCED LIMIT -->
-      <!--<limit effort="0" lower="0.000" upper="3.900" velocity="2.000"/>--> <!-- Product specification - IRBT 4004/6004/7004 -->
+      <limit effort="0" lower="0.000" upper="3.900" velocity="2.000"/> <!-- Product specification - IRBT 4004/6004/7004 -->
+    </joint>
+    <joint name="${prefix}joint_belt_loop" type="prismatic">
+      <parent link="${prefix}track_right"/>
+      <child link="${prefix}belt_loop"/>
+      <origin xyz="-0.1 0 0" rpy="0 0 0"/>
+      <axis xyz="-1 0 0"/>
+      <limit effort="0" lower="0.000" upper="3.900" velocity="2.000"/>
+      <mimic joint="${prefix}joint_carriage" multiplier="0.5"/>
+    </joint>
+    <joint name="${prefix}joint_belt_0" type="prismatic">
+      <parent link="${prefix}track_right"/>
+      <child link="${prefix}belt_0"/>
+      <origin xyz="-0.1 0 0" rpy="0 0 0"/>
+      <axis xyz="-1 0 0"/>
+      <limit effort="0" lower="0.000" upper="3.900" velocity="2.000"/>
+      <mimic joint="${prefix}joint_carriage" multiplier="0.5"/>
+    </joint>
+    <joint name="${prefix}joint_belt_1" type="prismatic">
+      <parent link="${prefix}track_right"/>
+      <child link="${prefix}belt_1"/>
+      <origin xyz="-0.1 0 0" rpy="0 0 0"/>
+      <axis xyz="-1 0 0"/>
+      <limit effort="0" lower="0.000" upper="3.900" velocity="2.000"/>
+      <mimic joint="${prefix}joint_carriage" multiplier="0.625"/>
+    </joint>
+    <joint name="${prefix}joint_belt_2" type="prismatic">
+      <parent link="${prefix}track_right"/>
+      <child link="${prefix}belt_2"/>
+      <origin xyz="-0.1 0 0" rpy="0 0 0"/>
+      <axis xyz="-1 0 0"/>
+      <limit effort="0" lower="0.000" upper="3.900" velocity="2.000"/>
+      <mimic joint="${prefix}joint_carriage" multiplier="0.75"/>
+    </joint>
+    <joint name="${prefix}joint_belt_3" type="prismatic">
+      <parent link="${prefix}track_right"/>
+      <child link="${prefix}belt_3"/>
+      <origin xyz="-0.1 0 0" rpy="0 0 0"/>
+      <axis xyz="-1 0 0"/>
+      <limit effort="0" lower="0.000" upper="3.900" velocity="2.000"/>
+      <mimic joint="${prefix}joint_carriage" multiplier="0.875"/>
+    </joint>
+    <joint name="${prefix}joint_belt_4" type="prismatic">
+      <parent link="${prefix}track_right"/>
+      <child link="${prefix}belt_4"/>
+      <origin xyz="-0.1 0 0" rpy="0 0 0"/>
+      <axis xyz="-1 0 0"/>
+      <limit effort="0" lower="0.500" upper="3.900" velocity="2.000"/>
+      <mimic joint="${prefix}joint_carriage" multiplier="1.0"/>
     </joint>
     <!-- Robot interface point -->

Commit message: update origins

File: abb_irbt4004_support/urdf/irbt4004_macro.xacro (robot description, xacro)
@@ -252,5 +252,5 @@
       <parent link="${prefix}track_left"/>
       <child link="${prefix}belt_loop"/>
-      <origin xyz="0 0 0" rpy="0 0 0"/>
+      <origin xyz="0.35 0 0" rpy="0 0 0"/>
       <axis xyz="1 0 0"/>
       <limit effort="0" lower="0.000" upper="3.900" velocity="2.000"/>
@@ -301,6 +301,7 @@
       <parent link="${prefix}carriage"/>
       <child link="${prefix}carriage_interface"/>
-      <origin xyz="0.3955 0.560 0.3745" rpy="0 0 1.57079632" />
-    </joint>
+      <origin xyz="0.3955 0.560 0.3745" rpy="0 0 1.57079632" /> <!-- 650-254=396 -->
+    </joint>
+<!--          <origin xyz="0.3955 0.560 0.3745" rpy="0 0 1.57079632" />-->
     <!-- end of joint list -->
   </xacro:macro>

File: abb_irbt4004_support/urdf/irbt4004r_macro.xacro (robot description, xacro)
@@ -89,5 +89,5 @@
     <link name="${prefix}carriage">
       <visual>
-      <origin xyz="-0.5 0 0" rpy="0 0 0"/>
+      <origin xyz="-0.6 0 0" rpy="0 0 0"/>
         <geometry>
           <mesh filename="package://abb_irbt4004_support/meshes/irbt4004/visual/Carriage_right.stl"/>
@@ -96,5 +96,5 @@
       </visual>
       <collision>
-        <origin xyz="-0.5 0 0" rpy="0 0 0"/>
+        <origin xyz="-0.6 0 0" rpy="0 0 0"/>
         <geometry>
           <mesh filename="package://abb_irbt4004_support/meshes/irbt4004/collision/Carriage_right.stl"/>
@@ -105,5 +105,5 @@
     <link name="${prefix}belt_loop">
       <visual>
-      <origin xyz="-0.5 0 0" rpy="0 0 0"/>
+      <origin xyz="-0.6 0 0" rpy="0 0 0"/>
         <geometry>
           <mesh filename="package://abb_irbt4004_support/meshes/irbt4004/visual/Belt_right_loop.stl"/>
@@ -112,5 +112,5 @@
       </visual>
       <collision>
-        <origin xyz="-0.5 0 0" rpy="0 0 0"/>
+        <origin xyz="-0.6 0 0" rpy="0 0 0"/>
         <geometry>
           <mesh filename="package://abb_irbt4004_support/meshes/irbt4004/collision/Belt_right_loop.stl"/>
@@ -121,12 +121,12 @@
     <link name="${prefix}belt_0">
       <visual>
-      <origin xyz="-0.5 0 0" rpy="0 0 0"/>
-        <geometry>
-          <mesh filename="package://abb_irbt4004_support/meshes/irbt4004/visual/Belt_right_ext.stl"/>
-        </geometry>
-        <xacro:material_abb_dark_gray />
-      </visual>
-      <collision>
-        <origin xyz="-0.5 0 0" rpy="0 0 0"/>
+      <origin xyz="-0.6 0 0" rpy="0 0 0"/>
+        <geometry>
+          <mesh filename="package://abb_irbt4004_support/meshes/irbt4004/visual/Belt_right_ext.stl"/>
+        </geometry>
+        <xacro:material_abb_dark_gray />
+      </visual>
+      <collision>
+        <origin xyz="-0.6 0 0" rpy="0 0 0"/>
         <geometry>
           <mesh filename="package://abb_irbt4004_support/meshes/irbt4004/collision/Belt_right_ext.stl"/>
@@ -137,12 +137,12 @@
     <link name="${prefix}belt_1">
       <visual>
-      <origin xyz="-0.5 0 0" rpy="0 0 0"/>
-        <geometry>
-          <mesh filename="package://abb_irbt4004_support/meshes/irbt4004/visual/Belt_right_ext.stl"/>
-        </geometry>
-        <xacro:material_abb_dark_gray />
-      </visual>
-      <collision>
-        <origin xyz="-0.5 0 0" rpy="0 0 0"/>
+      <origin xyz="-0.6 0 0" rpy="0 0 0"/>
+        <geometry>
+          <mesh filename="package://abb_irbt4004_support/meshes/irbt4004/visual/Belt_right_ext.stl"/>
+        </geometry>
+        <xacro:material_abb_dark_gray />
+      </visual>
+      <collision>
+        <origin xyz="-0.6 0 0" rpy="0 0 0"/>
         <geometry>
           <mesh filename="package://abb_irbt4004_support/meshes/irbt4004/collision/Belt_right_ext.stl"/>
@@ -153,12 +153,12 @@
     <link name="${prefix}belt_2">
       <visual>
-      <origin xyz="-0.5 0 0" rpy="0 0 0"/>
-        <geometry>
-          <mesh filename="package://abb_irbt4004_support/meshes/irbt4004/visual/Belt_right_ext.stl"/>
-        </geometry>
-        <xacro:material_abb_dark_gray />
-      </visual>
-      <collision>
-        <origin xyz="-0.5 0 0" rpy="0 0 0"/>
+      <origin xyz="-0.6 0 0" rpy="0 0 0"/>
+        <geometry>
+          <mesh filename="package://abb_irbt4004_support/meshes/irbt4004/visual/Belt_right_ext.stl"/>
+        </geometry>
+        <xacro:material_abb_dark_gray />
+      </visual>
+      <collision>
+        <origin xyz="-0.6 0 0" rpy="0 0 0"/>
         <geometry>
           <mesh filename="package://abb_irbt4004_support/meshes/irbt4004/collision/Belt_right_ext.stl"/>
@@ -169,12 +169,12 @@
     <link name="${prefix}belt_3">
       <visual>
-      <origin xyz="-0.5 0 0" rpy="0 0 0"/>
-        <geometry>
-          <mesh filename="package://abb_irbt4004_support/meshes/irbt4004/visual/Belt_right_ext.stl"/>
-        </geometry>
-        <xacro:material_abb_dark_gray />
-      </visual>
-      <collision>
-        <origin xyz="-0.5 0 0" rpy="0 0 0"/>
+      <origin xyz="-0.6 0 0" rpy="0 0 0"/>
+        <geometry>
+          <mesh filename="package://abb_irbt4004_support/meshes/irbt4004/visual/Belt_right_ext.stl"/>
+        </geometry>
+        <xacro:material_abb_dark_gray />
+      </visual>
+      <collision>
+        <origin xyz="-0.6 0 0" rpy="0 0 0"/>
         <geometry>
           <mesh filename="package://abb_irbt4004_support/meshes/irbt4004/collision/Belt_right_ext.stl"/>
@@ -185,12 +185,12 @@
     <link name="${prefix}belt_4">
       <visual>
-      <origin xyz="-0.5 0 0" rpy="0 0 0"/>
-        <geometry>
-          <mesh filename="package://abb_irbt4004_support/meshes/irbt4004/visual/Belt_right_ext.stl"/>
-        </geometry>
-        <xacro:material_abb_dark_gray />
-      </visual>
-      <collision>
-        <origin xyz="-0.5 0 0" rpy="0 0 0"/>
+      <origin xyz="-0.6 0 0" rpy="0 0 0"/>
+        <geometry>
+          <mesh filename="package://abb_irbt4004_support/meshes/irbt4004/visual/Belt_right_ext.stl"/>
+        </geometry>
+        <xacro:material_abb_dark_gray />
+      </visual>
+      <collision>
+        <origin xyz="-0.6 0 0" rpy="0 0 0"/>
         <geometry>
           <mesh filename="package://abb_irbt4004_support/meshes/irbt4004/collision/Belt_right_ext.stl"/>
@@ -226,5 +226,5 @@
       <parent link="${prefix}track_right"/>
       <child link="${prefix}carriage"/>
-      <origin xyz="-0.1 0 0" rpy="0 0 0"/>
+      <origin xyz="0 0 0" rpy="0 0 0"/>
       <axis xyz="-1 0 0"/>
       <limit effort="0" lower="0.000" upper="3.900" velocity="2.000"/> <!-- Product specification - IRBT 4004/6004/7004 -->
@@ -233,5 +233,5 @@
       <parent link="${prefix}track_right"/>
       <child link="${prefix}belt_loop"/>
-      <origin xyz="-0.1 0 0" rpy="0 0 0"/>
+      <origin xyz=" -0.35 0 0" rpy="0 0 0"/>
       <axis xyz="-1 0 0"/>
       <limit effort="0" lower="0.000" upper="3.900" velocity="2.000"/>
@@ -241,5 +241,5 @@
       <parent link="${prefix}track_right"/>
       <child link="${prefix}belt_0"/>
-      <origin xyz="-0.1 0 0" rpy="0 0 0"/>
+      <origin xyz="0 0 0" rpy="0 0 0"/>
       <axis xyz="-1 0 0"/>
       <limit effort="0" lower="0.000" upper="3.900" velocity="2.000"/>
@@ -249,5 +249,5 @@
       <parent link="${prefix}track_right"/>
       <child link="${prefix}belt_1"/>
-      <origin xyz="-0.1 0 0" rpy="0 0 0"/>
+      <origin xyz="0 0 0" rpy="0 0 0"/>
       <axis xyz="-1 0 0"/>
       <limit effort="0" lower="0.000" upper="3.900" velocity="2.000"/>
@@ -257,5 +257,5 @@
       <parent link="${prefix}track_right"/>
       <child link="${prefix}belt_2"/>
-      <origin xyz="-0.1 0 0" rpy="0 0 0"/>
+      <origin xyz="0 0 0" rpy="0 0 0"/>
       <axis xyz="-1 0 0"/>
       <limit effort="0" lower="0.000" upper="3.900" velocity="2.000"/>
@@ -265,5 +265,5 @@
       <parent link="${prefix}track_right"/>
       <child link="${prefix}belt_3"/>
-      <origin xyz="-0.1 0 0" rpy="0 0 0"/>
+      <origin xyz="0 0 0" rpy="0 0 0"/>
       <axis xyz="-1 0 0"/>
       <limit effort="0" lower="0.000" upper="3.900" velocity="2.000"/>
@@ -273,5 +273,5 @@
       <parent link="${prefix}track_right"/>
       <child link="${prefix}belt_4"/>
-      <origin xyz="-0.1 0 0" rpy="0 0 0"/>
+      <origin xyz="0 0 0" rpy="0 0 0"/>
       <axis xyz="-1 0 0"/>
       <limit effort="0" lower="0.500" upper="3.900" velocity="2.000"/>
@@ -282,7 +282,8 @@
       <parent link="${prefix}carriage"/>
       <child link="${prefix}carriage_interface"/>
-      <origin xyz="-0.1045 0.560 0.3745" rpy="0 0 1.57079632" />
+      <origin xyz="-0.2045 0.560 0.3745" rpy="0 0 1.57079632" />
     </joint>
     <!-- end of joint list -->
+<!--<origin xyz="-0.1045 0.560 0.3745" rpy="0 0 1.57079632" />-->
   </xacro:macro>
 </robot>
