Commit message: irbt4004: new static belt collision model

File: abb_irbt4004_support/urdf/irbt4004_macro.xacro (robot description, xacro)
@@ -104,4 +104,13 @@
       </collision>
     </link>
+    <link name="${prefix}belt_collision">
+        <collision>
+            <origin xyz="1.85 -0.20 0.3" rpy="0 0 0"/>
+            <geometry>
+                <box size="5.80 0.40 0.6"/>
+            </geometry>
+            <xacro:material_abb_dark_gray />
+        </collision>
+    </link>
     <link name="${prefix}belt_loop">
       <visual>
@@ -112,5 +121,5 @@
         <xacro:material_abb_dark_gray />
       </visual>
-      <collision>
+<!--      <collision>
         <origin xyz="0 0 0" rpy="0 0 0"/>
         <geometry>
@@ -118,5 +127,5 @@
         </geometry>
         <xacro:material_abb_dark_gray />
-      </collision>
+      </collision>-->
     </link>
     <link name="${prefix}belt_0">
@@ -128,11 +137,11 @@
         <xacro:material_abb_dark_gray />
       </visual>
-      <collision>
-        <origin xyz="0 0 0" rpy="0 0 0"/>
-        <geometry>
-          <mesh filename="package://abb_irbt4004_support/meshes/irbt4004/collision/Belt_left_ext.stl"/>
-        </geometry>
-        <xacro:material_abb_dark_gray />
-      </collision>
+<!--      <collision>
+        <origin xyz="0 0 0" rpy="0 0 0"/>
+        <geometry>
+          <mesh filename="package://abb_irbt4004_support/meshes/irbt4004/collision/Belt_left_ext.stl"/>
+        </geometry>
+        <xacro:material_abb_dark_gray />
+      </collision>-->
     </link>
     <link name="${prefix}belt_1">
@@ -144,11 +153,11 @@
         <xacro:material_abb_dark_gray />
       </visual>
-      <collision>
-        <origin xyz="0 0 0" rpy="0 0 0"/>
-        <geometry>
-          <mesh filename="package://abb_irbt4004_support/meshes/irbt4004/collision/Belt_left_ext.stl"/>
-        </geometry>
-        <xacro:material_abb_dark_gray />
-      </collision>
+<!--      <collision>
+        <origin xyz="0 0 0" rpy="0 0 0"/>
+        <geometry>
+          <mesh filename="package://abb_irbt4004_support/meshes/irbt4004/collision/Belt_left_ext.stl"/>
+        </geometry>
+        <xacro:material_abb_dark_gray />
+      </collision>-->
     </link>
     <link name="${prefix}belt_2">
@@ -160,11 +169,11 @@
         <xacro:material_abb_dark_gray />
       </visual>
-      <collision>
-        <origin xyz="0 0 0" rpy="0 0 0"/>
-        <geometry>
-          <mesh filename="package://abb_irbt4004_support/meshes/irbt4004/collision/Belt_left_ext.stl"/>
-        </geometry>
-        <xacro:material_abb_dark_gray />
-      </collision>
+<!--      <collision>
+        <origin xyz="0 0 0" rpy="0 0 0"/>
+        <geometry>
+          <mesh filename="package://abb_irbt4004_support/meshes/irbt4004/collision/Belt_left_ext.stl"/>
+        </geometry>
+        <xacro:material_abb_dark_gray />
+      </collision>-->
     </link>
     <link name="${prefix}belt_3">
@@ -176,11 +185,11 @@
         <xacro:material_abb_dark_gray />
       </visual>
-      <collision>
-        <origin xyz="0 0 0" rpy="0 0 0"/>
-        <geometry>
-          <mesh filename="package://abb_irbt4004_support/meshes/irbt4004/collision/Belt_left_ext.stl"/>
-        </geometry>
-        <xacro:material_abb_dark_gray />
-      </collision>
+<!--      <collision>
+        <origin xyz="0 0 0" rpy="0 0 0"/>
+        <geometry>
+          <mesh filename="package://abb_irbt4004_support/meshes/irbt4004/collision/Belt_left_ext.stl"/>
+        </geometry>
+        <xacro:material_abb_dark_gray />
+      </collision>-->
     </link>
     <link name="${prefix}belt_4">
@@ -192,11 +201,11 @@
         <xacro:material_abb_dark_gray />
       </visual>
-      <collision>
-        <origin xyz="0 0 0" rpy="0 0 0"/>
-        <geometry>
-          <mesh filename="package://abb_irbt4004_support/meshes/irbt4004/collision/Belt_left_ext.stl"/>
-        </geometry>
-        <xacro:material_abb_dark_gray />
-      </collision>
+<!--      <collision>
+        <origin xyz="0 0 0" rpy="0 0 0"/>
+        <geometry>
+          <mesh filename="package://abb_irbt4004_support/meshes/irbt4004/collision/Belt_left_ext.stl"/>
+        </geometry>
+        <xacro:material_abb_dark_gray />
+      </collision>-->
     </link>
     <!--Right carriage-->
@@ -249,4 +258,9 @@
       <limit effort="0" lower="0.000" upper="3.900" velocity="2.000"/> <!-- Product specification - IRBT 4004/6004/7004 -->
     </joint>
+    <joint name="${prefix}joint_belt_collision" type="fixed">
+      <parent link="${prefix}track_left"/>
+      <child link="${prefix}belt_collision"/>
+      <origin xyz="0 0 0" rpy="0 0 0"/>
+    </joint>
     <joint name="${prefix}joint_belt_loop" type="prismatic">
       <parent link="${prefix}track_left"/>

File: abb_irbt4004_support/urdf/irbt4004r_macro.xacro (robot description, xacro)
@@ -103,4 +103,13 @@
       </collision>
     </link>
+    <link name="${prefix}belt_collision">
+        <collision>
+            <origin xyz="-1.85 -0.20 0.3" rpy="0 0 0"/>
+            <geometry>
+                <box size="5.80 0.40 0.6"/>
+            </geometry>
+            <xacro:material_abb_dark_gray />
+        </collision>
+    </link>
     <link name="${prefix}belt_loop">
       <visual>
@@ -111,5 +120,5 @@
         <xacro:material_abb_dark_gray />
       </visual>
-      <collision>
+<!--      <collision>
         <origin xyz="-0.6 0 0" rpy="0 0 0"/>
         <geometry>
@@ -117,5 +126,5 @@
         </geometry>
         <xacro:material_abb_dark_gray />
-      </collision>
+      </collision>-->
     </link>
     <link name="${prefix}belt_0">
@@ -127,11 +136,11 @@
         <xacro:material_abb_dark_gray />
       </visual>
-      <collision>
-        <origin xyz="-0.6 0 0" rpy="0 0 0"/>
-        <geometry>
-          <mesh filename="package://abb_irbt4004_support/meshes/irbt4004/collision/Belt_right_ext.stl"/>
-        </geometry>
-        <xacro:material_abb_dark_gray />
-      </collision>
+<!--      <collision>
+        <origin xyz="-0.6 0 0" rpy="0 0 0"/>
+        <geometry>
+          <mesh filename="package://abb_irbt4004_support/meshes/irbt4004/collision/Belt_right_ext.stl"/>
+        </geometry>
+        <xacro:material_abb_dark_gray />
+      </collision>-->
     </link>
     <link name="${prefix}belt_1">
@@ -143,11 +152,11 @@
         <xacro:material_abb_dark_gray />
       </visual>
-      <collision>
-        <origin xyz="-0.6 0 0" rpy="0 0 0"/>
-        <geometry>
-          <mesh filename="package://abb_irbt4004_support/meshes/irbt4004/collision/Belt_right_ext.stl"/>
-        </geometry>
-        <xacro:material_abb_dark_gray />
-      </collision>
+<!--      <collision>
+        <origin xyz="-0.6 0 0" rpy="0 0 0"/>
+        <geometry>
+          <mesh filename="package://abb_irbt4004_support/meshes/irbt4004/collision/Belt_right_ext.stl"/>
+        </geometry>
+        <xacro:material_abb_dark_gray />
+      </collision>-->
     </link>
     <link name="${prefix}belt_2">
@@ -159,11 +168,11 @@
         <xacro:material_abb_dark_gray />
       </visual>
-      <collision>
-        <origin xyz="-0.6 0 0" rpy="0 0 0"/>
-        <geometry>
-          <mesh filename="package://abb_irbt4004_support/meshes/irbt4004/collision/Belt_right_ext.stl"/>
-        </geometry>
-        <xacro:material_abb_dark_gray />
-      </collision>
+<!--      <collision>
+        <origin xyz="-0.6 0 0" rpy="0 0 0"/>
+        <geometry>
+          <mesh filename="package://abb_irbt4004_support/meshes/irbt4004/collision/Belt_right_ext.stl"/>
+        </geometry>
+        <xacro:material_abb_dark_gray />
+      </collision>-->
     </link>
     <link name="${prefix}belt_3">
@@ -175,11 +184,11 @@
         <xacro:material_abb_dark_gray />
       </visual>
-      <collision>
-        <origin xyz="-0.6 0 0" rpy="0 0 0"/>
-        <geometry>
-          <mesh filename="package://abb_irbt4004_support/meshes/irbt4004/collision/Belt_right_ext.stl"/>
-        </geometry>
-        <xacro:material_abb_dark_gray />
-      </collision>
+<!--      <collision>
+        <origin xyz="-0.6 0 0" rpy="0 0 0"/>
+        <geometry>
+          <mesh filename="package://abb_irbt4004_support/meshes/irbt4004/collision/Belt_right_ext.stl"/>
+        </geometry>
+        <xacro:material_abb_dark_gray />
+      </collision>-->
     </link>
     <link name="${prefix}belt_4">
@@ -191,11 +200,11 @@
         <xacro:material_abb_dark_gray />
       </visual>
-      <collision>
-        <origin xyz="-0.6 0 0" rpy="0 0 0"/>
-        <geometry>
-          <mesh filename="package://abb_irbt4004_support/meshes/irbt4004/collision/Belt_right_ext.stl"/>
-        </geometry>
-        <xacro:material_abb_dark_gray />
-      </collision>
+<!--      <collision>
+        <origin xyz="-0.6 0 0" rpy="0 0 0"/>
+        <geometry>
+          <mesh filename="package://abb_irbt4004_support/meshes/irbt4004/collision/Belt_right_ext.stl"/>
+        </geometry>
+        <xacro:material_abb_dark_gray />
+      </collision>-->
     </link>
     <link name="${prefix}carriage_interface"/>
@@ -229,4 +238,9 @@
       <axis xyz="-1 0 0"/>
       <limit effort="0" lower="0.000" upper="3.900" velocity="2.000"/> <!-- Product specification - IRBT 4004/6004/7004 -->
+    </joint>
+    <joint name="${prefix}joint_belt_collision" type="fixed">
+      <parent link="${prefix}track_right"/>
+      <child link="${prefix}belt_collision"/>
+      <origin xyz="0 0 0" rpy="0 0 0"/>
     </joint>
     <joint name="${prefix}joint_belt_loop" type="prismatic">
