Commit message: irbt4004 - changed limits

File: abb_irb4400_support/urdf/irb4400_60_macro.xacro (robot description, xacro)
@@ -159,5 +159,6 @@
       <child link="${prefix}link_6"/>
       <axis xyz="1 0 0"/>
-      <limit effort="0" lower="-6.9813" upper="6.9813" velocity="5.7596"/>
+      <limit effort="0" lower="-3.1415" upper="3.1415" velocity="5.7596"/>  <!--reduced to 180deg-->
+<!--      <limit effort="0" lower="-6.9813" upper="6.9813" velocity="5.7596"/>--> <!--spec-->
     </joint>
     <joint name="${prefix}joint_6-tool0" type="fixed">

File: abb_irbt4004_support/urdf/irbt4004_macro.xacro (robot description, xacro)
@@ -151,5 +151,6 @@
       <origin xyz="0 0 0" rpy="0 0 0"/>
       <axis xyz="1 0 0"/>
-      <limit effort="0" lower="0.000" upper="3.900" velocity="2.000"/> <!-- Product specification - IRBT 4004/6004/7004 -->
+      <limit effort="0" lower="0.000" upper="3.400" velocity="2.000"/> <!-- REDUCED LIMIT -->
+      <!--<limit effort="0" lower="0.000" upper="3.900" velocity="2.000"/>--> <!-- Product specification - IRBT 4004/6004/7004 -->
     </joint>
     <!-- Robot interface point -->

File: abb_irbt4004_support/urdf/irbt4004r_macro.xacro (robot description, xacro)
@@ -132,5 +132,6 @@
       <origin xyz="-0.1 0 0" rpy="0 0 0"/>
       <axis xyz="-1 0 0"/>
-      <limit effort="0" lower="0.000" upper="3.900" velocity="2.000"/> <!-- Product specification - IRBT 4004/6004/7004 -->
+      <limit effort="0" lower="0.000" upper="3.400" velocity="2.000"/> <!-- REDUCED LIMIT -->
+      <!--<limit effort="0" lower="0.000" upper="3.900" velocity="2.000"/>--> <!-- Product specification - IRBT 4004/6004/7004 -->
     </joint>
     <!-- Robot interface point -->

Commit message: update limits

File: abb_irb4400_support/urdf/irb4400_60_macro.xacro (robot description, xacro)
@@ -137,5 +137,7 @@
       <child link="${prefix}link_3"/>
       <axis xyz="0 1 0"/>
-      <limit effort="0" lower="-1.0472" upper="1.1345" velocity="2.0944"/>
+      <limit effort="0" lower="-0.2" upper="1.1345" velocity="2.0944"/> <!--less than robotstudio to avoid out of range-->
+<!--      <limit effort="0" lower="-0.523599" upper="1.1345" velocity="2.0944"/>--> <!--robotstudio-->
+<!--      <limit effort="0" lower="-1.0472" upper="1.1345" velocity="2.0944"/> -->
     </joint>
     <joint name="${prefix}joint_4" type="revolute">

Commit message: irb_4400_60: updated collision mesh

File: abb_irb4400_support/urdf/irb4400_60_macro.xacro (robot description, xacro)
@@ -111,4 +111,36 @@
         <geometry>
           <mesh filename="package://abb_irb4400_support/meshes/irb4400_60/collision/link_6.stl"/>
+        </geometry>
+        <xacro:material_abb_yellow />
+      </collision>
+    </link>
+    <link name="${prefix}link_d1">
+      <visual>
+        <origin xyz="0 0 0" rpy="0 0 0"/>
+        <geometry>
+          <mesh filename="package://abb_irb4400_support/meshes/irb4400_60/visual/link_d1.stl"/>
+        </geometry>
+        <xacro:material_abb_orange />
+      </visual>
+      <collision>
+        <origin xyz="0 0 0" rpy="0 0 0"/>
+        <geometry>
+          <mesh filename="package://abb_irb4400_support/meshes/irb4400_60/collision/link_d1.stl"/>
+        </geometry>
+        <xacro:material_abb_yellow />
+      </collision>
+    </link>
+    <link name="${prefix}link_d2">
+      <visual>
+        <origin xyz="0 0 0" rpy="0 0 0"/>
+        <geometry>
+          <mesh filename="package://abb_irb4400_support/meshes/irb4400_60/visual/link_d2.stl"/>
+        </geometry>
+        <xacro:material_abb_orange />
+      </visual>
+      <collision>
+        <origin xyz="0 0 0" rpy="0 0 0"/>
+        <geometry>
+          <mesh filename="package://abb_irb4400_support/meshes/irb4400_60/collision/link_d2.stl"/>
         </geometry>
         <xacro:material_abb_yellow />
@@ -169,4 +201,18 @@
       <origin xyz="0.14 0 0" rpy="0 0 0"/>
     </joint>
+    <joint name="${prefix}joint_d2" type="continuous" >
+      <origin xyz="0 0 0" rpy="0 0 0"/>
+      <axis xyz="0 1 0"/>
+      <parent link="${prefix}link_2"/>
+      <child link="${prefix}link_d2"/>
+      <mimic joint="${prefix}joint_3" multiplier="1.0"/>
+    </joint>
+    <joint name="${prefix}joint_d1" type="continuous" >
+      <origin xyz="-0.3 0 0" rpy="0 0 0"/>
+      <axis xyz="0 1 0"/>
+      <parent link="${prefix}link_d2"/>
+      <child link="${prefix}link_d1"/>
+      <mimic joint="${prefix}joint_3" multiplier="-1.0"/>
+    </joint>
     <!-- end of joint list -->
     <!-- ROS base_link to ABB World Coordinates transform -->
